Commit message: resulting files

File: outputs/naogazeboarms.xacro (robot description, xacro)
@@ -4,6 +4,6 @@
 		<parent link="torso"/>
 		<child link="LShoulder"/>
-		<origin rpy="0 0 0" xyz="0 0 0"/>
-		<axis xyz="0 0 0"/>
+		<origin rpy="0 0 0" xyz="0 0.098 0.1"/>
+		<axis xyz="0 1.0 0"/>
 		<limit effort="1.2" lower="-2.08567" upper="2.08567" velocity="8.26797"/>
 	</joint>
@@ -11,11 +11,10 @@
 		<visual>
 			<geometry>
-				<mesh filename="file:///home/marguedas/.ros/nao_meshes/meshes/V40/visual/LShoulder.obj" scale="0 0 0"/>
-			</geometry>
-			<origin rpy="0 0 0" xyz="0 0 0"/>
-		</visual>
-		<collision>
-			<geometry>
-				<mesh filename="file:///home/marguedas/.ros/nao_meshes/meshes/V40/collision/LShoulder.ply" scale="0 0 0"/>
+				<mesh filename="file:///home/marguedas/.ros/nao_meshes/meshes/V40/visual/collada/LShoulder.dae" scale="0.1 0.1 0.1"/>
+			</geometry>
+		</visual>
+		<collision>
+			<geometry>
+				<mesh filename="file:///home/marguedas/.ros/nao_meshes/meshes/V40/visual/collada/LShoulder.dae" scale="0.1 0.1 0.1"/>
 			</geometry>
 		</collision>
@@ -23,5 +22,5 @@
 			<mass value="0.07504"/>
 			<inertia ixx="8.42843e-05" ixy="-2.02802e-06" ixz="2.338e-08" iyy="1.41556e-05" iyz="-1.972e-08" izz="8.64195e-05"/>
-			<origin rpy="0 0 0" xyz="0 0 0"/>
+			<origin rpy="0 0 0" xyz="-0.00165 -0.02663 0.00014"/>
 		</inertial>
 	</link>
@@ -30,5 +29,5 @@
 		<child link="LBicep"/>
 		<origin rpy="0 0 0" xyz="0 0 0"/>
-		<axis xyz="0 0 0"/>
+		<axis xyz="0 0 1.0"/>
 		<limit effort="1.2" lower="-0.314159" upper="1.32645" velocity="7.19407"/>
 	</joint>
@@ -36,11 +35,10 @@
 		<visual>
 			<geometry>
-				<mesh filename="file:///home/marguedas/.ros/nao_meshes/meshes/V40/visual/LBicep.obj" scale="0 0 0"/>
-			</geometry>
-			<origin rpy="0 0 0" xyz="0 0 0"/>
-		</visual>
-		<collision>
-			<geometry>
-				<mesh filename="file:///home/marguedas/.ros/nao_meshes/meshes/V40/collision/LBicep.ply" scale="0 0 0"/>
+				<mesh filename="file:///home/marguedas/.ros/nao_meshes/meshes/V40/visual/collada/LBicep.dae" scale="0.1 0.1 0.1"/>
+			</geometry>
+		</visual>
+		<collision>
+			<geometry>
+				<mesh filename="file:///home/marguedas/.ros/nao_meshes/meshes/V40/visual/collada/LBicep.dae" scale="0.1 0.1 0.1"/>
 			</geometry>
 		</collision>
@@ -48,5 +46,5 @@
 			<mass value="0.15777"/>
 			<inertia ixx="9.38999e-05" ixy="-4.71445e-05" ixz="-2.69947e-05" iyy="0.000371519" iyz="-2.45977e-06" izz="0.000341901"/>
-			<origin rpy="0 0 0" xyz="0 0 0"/>
+			<origin rpy="0 0 0" xyz="0.02455 0.00563 0.0033"/>
 		</inertial>
 	</link>
@@ -54,6 +52,6 @@
 		<parent link="LBicep"/>
 		<child link="LElbow"/>
-		<origin rpy="0 0 0" xyz="0 0 0"/>
-		<axis xyz="0 0 0"/>
+		<origin rpy="0 0 0" xyz="0.105 0.015 0"/>
+		<axis xyz="1.0 0 0"/>
 		<limit effort="1.2" lower="-2.08567" upper="2.08567" velocity="8.26797"/>
 	</joint>
@@ -62,5 +60,5 @@
 			<mass value="0.06483"/>
 			<inertia ixx="5.59715e-06" ixy="4.21e-09" ixz="4.319e-08" iyy="7.54331e-05" iyz="-1.84e-09" izz="7.64434e-05"/>
-			<origin rpy="0 0 0" xyz="0 0 0"/>
+			<origin rpy="0 0 0" xyz="-0.02744 0 -0.00014"/>
 		</inertial>
 	</link>
@@ -69,5 +67,5 @@
 		<child link="LForeArm"/>
 		<origin rpy="0 0 0" xyz="0 0 0"/>
-		<axis xyz="0 0 0"/>
+		<axis xyz="0 0 1.0"/>
 		<limit effort="1.2" lower="-1.54462" upper="-0.0349066" velocity="7.19407"/>
 	</joint>
@@ -75,11 +73,10 @@
 		<visual>
 			<geometry>
-				<mesh filename="file:///home/marguedas/.ros/nao_meshes/meshes/V40/visual/LForeArm.obj" scale="0 0 0"/>
-			</geometry>
-			<origin rpy="0 0 0" xyz="0 0 0"/>
-		</visual>
-		<collision>
-			<geometry>
-				<mesh filename="file:///home/marguedas/.ros/nao_meshes/meshes/V40/collision/LForeArm.ply" scale="0 0 0"/>
+				<mesh filename="file:///home/marguedas/.ros/nao_meshes/meshes/V40/visual/collada/LForeArm.dae" scale="0.1 0.1 0.1"/>
+			</geometry>
+		</visual>
+		<collision>
+			<geometry>
+				<mesh filename="file:///home/marguedas/.ros/nao_meshes/meshes/V40/visual/collada/LForeArm.dae" scale="0.1 0.1 0.1"/>
 			</geometry>
 		</collision>
@@ -87,5 +84,5 @@
 			<mass value="0.07761"/>
 			<inertia ixx="2.53322e-05" ixy="-2.34271e-06" ixz="7.459e-08" iyy="8.91322e-05" iyz="-2.655e-08" izz="8.72873e-05"/>
-			<origin rpy="0 0 0" xyz="0 0 0"/>
+			<origin rpy="0 0 0" xyz="0.02556 0.00281 0.00076"/>
 		</inertial>
 	</link>
@@ -93,6 +90,6 @@
 		<parent link="LForeArm"/>
 		<child link="l_wrist"/>
-		<origin rpy="0 0 0" xyz="0 0 0"/>
-		<axis xyz="0 0 0"/>
+		<origin rpy="0 0 0" xyz="0.05595 0 0"/>
+		<axis xyz="1.0 0 0"/>
 		<limit effort="0.76" lower="-1.82387" upper="1.82387" velocity="24.6229"/>
 	</joint>
@@ -100,11 +97,10 @@
 		<visual>
 			<geometry>
-				<mesh filename="file:///home/marguedas/.ros/nao_meshes/meshes/V40/visual/l_wrist.obj" scale="0 0 0"/>
-			</geometry>
-			<origin rpy="0 0 0" xyz="0 0 0"/>
-		</visual>
-		<collision>
-			<geometry>
-				<mesh filename="file:///home/marguedas/.ros/nao_meshes/meshes/V40/collision/l_wrist.ply" scale="0 0 0"/>
+				<mesh filename="file:///home/marguedas/.ros/nao_meshes/meshes/V40/visual/collada/l_wrist.dae" scale="0.1 0.1 0.1"/>
+			</geometry>
+		</visual>
+		<collision>
+			<geometry>
+				<mesh filename="file:///home/marguedas/.ros/nao_meshes/meshes/V40/visual/collada/l_wrist.dae" scale="0.1 0.1 0.1"/>
 			</geometry>
 		</collision>
@@ -112,21 +108,21 @@
 			<mass value="0.18533"/>
 			<inertia ixx="7.05493e-05" ixy="5.71599e-06" ixz="-2.24744e-05" iyy="0.000356062" iyz="3.17771e-06" izz="0.000351919"/>
-			<origin rpy="0 0 0" xyz="0 0 0"/>
-		</inertial>
-	</link>
-	<joint name="LHand" type="revolute">
+			<origin rpy="0 0 0" xyz="0.03434 -0.00088 0.00308"/>
+		</inertial>
+	</link>
+	<joint name="LHand" type="fixed">
 		<parent link="l_wrist"/>
 		<child link="l_gripper"/>
-		<origin rpy="0 0 0" xyz="0 0 0"/>
+		<origin rpy="0 0 0" xyz="0.05775 0 -0.01231"/>
 	</joint>
 	<link name="l_gripper">
 		<visual>
 			<geometry>
-				<mesh filename="file:///home/marguedas/.ros/nao_meshes/meshes/V40/visual/l_gripper.obj" scale="0 0 0"/>
-			</geometry>
-		</visual>
-		<collision>
-			<geometry>
-				<mesh filename="file:///home/marguedas/.ros/nao_meshes/meshes/V40/collision/l_gripper.ply" scale="0 0 0"/>
+				<mesh filename="file:///home/marguedas/.ros/nao_meshes/meshes/V40/visual/collada/l_gripper.dae" scale="0.1 0.1 0.1"/>
+			</geometry>
+		</visual>
+		<collision>
+			<geometry>
+				<mesh filename="file:///home/marguedas/.ros/nao_meshes/meshes/V40/visual/collada/l_gripper.dae" scale="0.1 0.1 0.1"/>
 			</geometry>
 		</collision>
@@ -135,6 +131,6 @@
 		<parent link="torso"/>
 		<child link="RShoulder"/>
-		<origin rpy="0 0 0" xyz="0 0 0"/>
-		<axis xyz="0 0 0"/>
+		<origin rpy="0 0 0" xyz="0 -0.098 0.1"/>
+		<axis xyz="0 1.0 0"/>
 		<limit effort="1.2" lower="-2.08567" upper="2.08567" velocity="8.26797"/>
 	</joint>
@@ -142,11 +138,10 @@
 		<visual>
 			<geometry>
-				<mesh filename="file:///home/marguedas/.ros/nao_meshes/meshes/V40/visual/RShoulder.obj" scale="0 0 0"/>
-			</geometry>
-			<origin rpy="0 0 0" xyz="0 0 0"/>
-		</visual>
-		<collision>
-			<geometry>
-				<mesh filename="file:///home/marguedas/.ros/nao_meshes/meshes/V40/collision/RShoulder.ply" scale="0 0 0"/>
+				<mesh filename="file:///home/marguedas/.ros/nao_meshes/meshes/V40/visual/collada/RShoulder.dae" scale="0.1 0.1 0.1"/>
+			</geometry>
+		</visual>
+		<collision>
+			<geometry>
+				<mesh filename="file:///home/marguedas/.ros/nao_meshes/meshes/V40/visual/collada/RShoulder.dae" scale="0.1 0.1 0.1"/>
 			</geometry>
 		</collision>
@@ -154,5 +149,5 @@
 			<mass value="0.07504"/>
 			<inertia ixx="8.42843e-05" ixy="2.02802e-06" ixz="2.338e-08" iyy="1.41556e-05" iyz="1.972e-08" izz="8.64195e-05"/>
-			<origin rpy="0 0 0" xyz="0 0 0"/>
+			<origin rpy="0 0 0" xyz="-0.00165 0.02663 0.00014"/>
 		</inertial>
 	</link>
@@ -161,5 +156,5 @@
 		<child link="RBicep"/>
 		<origin rpy="0 0 0" xyz="0 0 0"/>
-		<axis xyz="0 0 0"/>
+		<axis xyz="0 0 1.0"/>
 		<limit effort="1.2" lower="-1.32645" upper="0.314159" velocity="7.19407"/>
 	</joint>
@@ -167,11 +162,10 @@
 		<visual>
 			<geometry>
-				<mesh filename="file:///home/marguedas/.ros/nao_meshes/meshes/V40/visual/RBicep.obj" scale="0 0 0"/>
-			</geometry>
-			<origin rpy="0 0 0" xyz="0 0 0"/>
-		</visual>
-		<collision>
-			<geometry>
-				<mesh filename="file:///home/marguedas/.ros/nao_meshes/meshes/V40/collision/RBicep.ply" scale="0 0 0"/>
+				<mesh filename="file:///home/marguedas/.ros/nao_meshes/meshes/V40/visual/collada/RBicep.dae" scale="0.1 0.1 0.1"/>
+			</geometry>
+		</visual>
+		<collision>
+			<geometry>
+				<mesh filename="file:///home/marguedas/.ros/nao_meshes/meshes/V40/visual/collada/RBicep.dae" scale="0.1 0.1 0.1"/>
 			</geometry>
 		</collision>
@@ -179,5 +173,5 @@
 			<mass value="0.15777"/>
 			<inertia ixx="0.00011012" ixy="7.66913e-05" ixz="-2.60461e-05" iyy="0.000367577" iyz="1.20983e-05" izz="0.000354618"/>
-			<origin rpy="0 0 0" xyz="0 0 0"/>
+			<origin rpy="0 0 0" xyz="0.02455 -0.00563 0.0033"/>
 		</inertial>
 	</link>
@@ -185,6 +179,6 @@
 		<parent link="RBicep"/>
 		<child link="RElbow"/>
-		<origin rpy="0 0 0" xyz="0 0 0"/>
-		<axis xyz="0 0 0"/>
+		<origin rpy="0 0 0" xyz="0.105 -0.015 0"/>
+		<axis xyz="1.0 0 0"/>
 		<limit effort="1.2" lower="-2.08567" upper="2.08567" velocity="8.26797"/>
 	</joint>
@@ -193,5 +187,5 @@
 			<mass value="0.06483"/>
 			<inertia ixx="5.59715e-06" ixy="4.21e-09" ixz="4.319e-08" iyy="7.54331e-05" iyz="-1.84e-09" izz="7.64434e-05"/>
-			<origin rpy="0 0 0" xyz="0 0 0"/>
+			<origin rpy="0 0 0" xyz="-0.02744 0 -0.00014"/>
 		</inertial>
 	</link>
@@ -200,5 +194,5 @@
 		<child link="RForeArm"/>
 		<origin rpy="0 0 0" xyz="0 0 0"/>
-		<axis xyz="0 0 0"/>
+		<axis xyz="0 0 1.0"/>
 		<limit effort="1.2" lower="0.0349066" upper="1.54462" velocity="7.19407"/>
 	</joint>
@@ -206,11 +200,10 @@
 		<visual>
 			<geometry>
-				<mesh filename="file:///home/marguedas/.ros/nao_meshes/meshes/V40/visual/RForeArm.obj" scale="0 0 0"/>
-			</geometry>
-			<origin rpy="0 0 0" xyz="0 0 0"/>
-		</visual>
-		<collision>
-			<geometry>
-				<mesh filename="file:///home/marguedas/.ros/nao_meshes/meshes/V40/collision/RForeArm.ply" scale="0 0 0"/>
+				<mesh filename="file:///home/marguedas/.ros/nao_meshes/meshes/V40/visual/collada/RForeArm.dae" scale="0.1 0.1 0.1"/>
+			</geometry>
+		</visual>
+		<collision>
+			<geometry>
+				<mesh filename="file:///home/marguedas/.ros/nao_meshes/meshes/V40/visual/collada/RForeArm.dae" scale="0.1 0.1 0.1"/>
 			</geometry>
 		</collision>
@@ -218,5 +211,5 @@
 			<mass value="0.07761"/>
 			<inertia ixx="2.53907e-05" ixy="2.33243e-06" ixz="-6.0117e-07" iyy="8.92204e-05" iyz="2.694e-08" izz="8.72484e-05"/>
-			<origin rpy="0 0 0" xyz="0 0 0"/>
+			<origin rpy="0 0 0" xyz="0.02556 -0.00281 0.00076"/>
 		</inertial>
 	</link>
@@ -224,6 +217,6 @@
 		<parent link="RForeArm"/>
 		<child link="r_wrist"/>
-		<origin rpy="0 0 0" xyz="0 0 0"/>
-		<axis xyz="0 0 0"/>
+		<origin rpy="0 0 0" xyz="0.05595 0 0"/>
+		<axis xyz="1.0 0 0"/>
 		<limit effort="0.76" lower="-1.82387" upper="1.82387" velocity="24.6229"/>
 	</joint>
@@ -231,11 +224,10 @@
 		<visual>
 			<geometry>
-				<mesh filename="file:///home/marguedas/.ros/nao_meshes/meshes/V40/visual/r_wrist.obj" scale="0 0 0"/>
-			</geometry>
-			<origin rpy="0 0 0" xyz="0 0 0"/>
-		</visual>
-		<collision>
-			<geometry>
-				<mesh filename="file:///home/marguedas/.ros/nao_meshes/meshes/V40/collision/r_wrist.ply" scale="0 0 0"/>
+				<mesh filename="file:///home/marguedas/.ros/nao_meshes/meshes/V40/visual/collada/r_wrist.dae" scale="0.1 0.1 0.1"/>
+			</geometry>
+		</visual>
+		<collision>
+			<geometry>
+				<mesh filename="file:///home/marguedas/.ros/nao_meshes/meshes/V40/visual/collada/r_wrist.dae" scale="0.1 0.1 0.1"/>
 			</geometry>
 		</collision>
@@ -243,21 +235,21 @@
 			<mass value="0.18533"/>
 			<inertia ixx="7.05493e-05" ixy="5.71599e-06" ixz="-2.24744e-05" iyy="0.000356062" iyz="3.17771e-06" izz="0.000351919"/>
-			<origin rpy="0 0 0" xyz="0 0 0"/>
-		</inertial>
-	</link>
-	<joint name="RHand" type="revolute">
+			<origin rpy="0 0 0" xyz="0.03434 0.00088 0.00308"/>
+		</inertial>
+	</link>
+	<joint name="RHand" type="fixed">
 		<parent link="r_wrist"/>
 		<child link="r_gripper"/>
-		<origin rpy="0 0 0" xyz="0 0 0"/>
+		<origin rpy="0 0 0" xyz="0.05775 0 -0.01231"/>
 	</joint>
 	<link name="r_gripper">
 		<visual>
 			<geometry>
-				<mesh filename="file:///home/marguedas/.ros/nao_meshes/meshes/V40/visual/r_gripper.obj" scale="0 0 0"/>
-			</geometry>
-		</visual>
-		<collision>
-			<geometry>
-				<mesh filename="file:///home/marguedas/.ros/nao_meshes/meshes/V40/collision/r_gripper.ply" scale="0 0 0"/>
+				<mesh filename="file:///home/marguedas/.ros/nao_meshes/meshes/V40/visual/collada/r_gripper.dae" scale="0.1 0.1 0.1"/>
+			</geometry>
+		</visual>
+		<collision>
+			<geometry>
+				<mesh filename="file:///home/marguedas/.ros/nao_meshes/meshes/V40/visual/collada/r_gripper.dae" scale="0.1 0.1 0.1"/>
 			</geometry>
 		</collision>

File: outputs/naogazebohead.xacro (robot description, xacro)
@@ -4,6 +4,6 @@
 		<parent link="torso"/>
 		<child link="Neck"/>
-		<origin rpy="0 0 0" xyz="0 0 0"/>
-		<axis xyz="0 0 0"/>
+		<origin rpy="0 0 0" xyz="0 0 0.1265"/>
+		<axis xyz="0 0 1.0"/>
 		<limit effort="1.2" lower="-2.08567" upper="2.08567" velocity="8.26797"/>
 	</joint>
@@ -11,11 +11,10 @@
 		<visual>
 			<geometry>
-				<mesh filename="file:///home/marguedas/.ros/nao_meshes/meshes/V40/visual/Neck.obj" scale="0 0 0"/>
+				<mesh filename="file:///home/marguedas/.ros/nao_meshes/meshes/V40/visual/collada/Neck.dae" scale="0.1 0.1 0.1"/>
 			</geometry>
-			<origin rpy="0 0 0" xyz="0 0 0"/>
 		</visual>
 		<collision>
 			<geometry>
-				<mesh filename="file:///home/marguedas/.ros/nao_meshes/meshes/V40/collision/Neck.ply" scale="0 0 0"/>
+				<mesh filename="file:///home/marguedas/.ros/nao_meshes/meshes/V40/visual/collada/Neck.dae" scale="0.1 0.1 0.1"/>
 			</geometry>
 		</collision>
@@ -23,5 +22,5 @@
 			<mass value="0.06442"/>
 			<inertia ixx="7.4993e-05" ixy="1.57e-09" ixz="-1.834e-08" iyy="7.6e-05" iyz="-5.295e-08" izz="5.53373e-06"/>
-			<origin rpy="0 0 0" xyz="0 0 0"/>
+			<origin rpy="0 0 0" xyz="-1e-05 0 -0.02742"/>
 		</inertial>
 	</link>
@@ -30,5 +29,5 @@
 		<child link="Head"/>
 		<origin rpy="0 0 0" xyz="0 0 0"/>
-		<axis xyz="0 0 0"/>
+		<axis xyz="0 1.0 0"/>
 		<limit effort="1.2" lower="-0.671952" upper="0.514872" velocity="7.19407"/>
 	</joint>
@@ -36,11 +35,10 @@
 		<visual>
 			<geometry>
-				<mesh filename="file:///home/marguedas/.ros/nao_meshes/meshes/V40/visual/Head.obj" scale="0 0 0"/>
+				<mesh filename="file:///home/marguedas/.ros/nao_meshes/meshes/V40/visual/collada/Head.dae" scale="0.1 0.1 0.1"/>
 			</geometry>
-			<origin rpy="0 0 0" xyz="0 0 0"/>
 		</visual>
 		<collision>
 			<geometry>
-				<mesh filename="file:///home/marguedas/.ros/nao_meshes/meshes/V40/collision/Head.ply" scale="0 0 0"/>
+				<mesh filename="file:///home/marguedas/.ros/nao_meshes/meshes/V40/visual/collada/Head.dae" scale="0.1 0.1 0.1"/>
 			</geometry>
 		</collision>
@@ -48,5 +46,5 @@
 			<mass value="0.60533"/>
 			<inertia ixx="0.0026313" ixy="8.78814e-06" ixz="4.09847e-05" iyy="0.00249112" iyz="-2.99579e-05" izz="0.000985736"/>
-			<origin rpy="0 0 0" xyz="0 0 0"/>
+			<origin rpy="0 0 0" xyz="-0.00112 0 0.05258"/>
 		</inertial>
 	</link>
@@ -54,5 +52,5 @@
 		<parent link="Head"/>
 		<child link="CameraTop_frame"/>
-		<origin rpy="0 0 0" xyz="0 0 0"/>
+		<origin rpy="0 0 0" xyz="0.0539 0 0.0679"/>
 	</joint>
 	<link name="CameraTop_frame"/>

File: outputs/naogazebotorso.xacro (robot description, xacro)
@@ -10,11 +10,10 @@
 		<visual>
 			<geometry>
-				<mesh filename="file:///home/marguedas/.ros/nao_meshes/meshes/V40/visual/torso.obj" scale="0 0 0"/>
+				<mesh filename="file:///home/marguedas/.ros/nao_meshes/meshes/V40/visual/collada/torso.dae" scale="0.1 0.1 0.1"/>
 			</geometry>
-			<origin rpy="0 0 0" xyz="0 0 0"/>
 		</visual>
 		<collision>
 			<geometry>
-				<mesh filename="file:///home/marguedas/.ros/nao_meshes/meshes/V40/collision/torso.ply" scale="0 0 0"/>
+				<mesh filename="file:///home/marguedas/.ros/nao_meshes/meshes/V40/visual/collada/torso.dae" scale="0.1 0.1 0.1"/>
 			</geometry>
 		</collision>
@@ -22,5 +21,5 @@
 			<mass value="1.04956"/>
 			<inertia ixx="0.00506234" ixy="1.43116e-05" ixz="0.000155191" iyy="0.00488014" iyz="-2.70793e-05" izz="0.0016103"/>
-			<origin rpy="0 0 0" xyz="0 0 0"/>
+			<origin rpy="0 0 0" xyz="-0.00413 0 0.04342"/>
 		</inertial>
 	</link>

File: outputs/naorobotrviz.urdf (robot description, URDF)
Before this commit: robot naoH25V40, 30 links, 29 joints
Links:
- link Head: geometry visual mesh filename=file:///nao/V40/HeadPitch.mesh scale=0.001 0.001 0.001
- link LBicep: geometry visual mesh filename=file:///home/marguedas/.ros/nao_meshes/meshes/V40/visual/co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 scale=0.1 0.1 0.1
- link LForeArm: geometry visual mesh filename=file:///home/marguedas/.ros/nao_meshes/meshes/V40/visual/co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 scale=0.1 0.1 0.1
- link LHip: geometry visual mesh filename=file:///home/marguedas/.ros/nao_meshes/meshes/V40/visual/co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 scale=0.1 0.1 0.1
- link LPelvis: geometry visual mesh filename=file:///home/marguedas/.ros/nao_meshes/meshes/V40/visual/co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 scale=0.1 0.1 0.1
- link LShoulder: geometry visual mesh filename=file:///home/marguedas/.ros/nao_meshes/meshes/V40/visual/co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 scale=0.1 0.1 0.1
- link LThigh: geometry visual mesh filename=file:///home/marguedas/.ros/nao_meshes/meshes/V40/visual/co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 scale=0.1 0.1 0.1
- link LTibia: geometry visual mesh filename=file:///home/marguedas/.ros/nao_meshes/meshes/V40/visual/co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 scale=0.1 0.1 0.1
- link Neck: geometry visual mesh filename=file:///home/marguedas/.ros/nao_meshes/meshes/V40/visual/co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 scale=0.1 0.1 0.1
- link RBicep: geometry visual mesh filename=file:///home/marguedas/.ros/nao_meshes/meshes/V40/visual/co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 scale=0.1 0.1 0.1
- link RForeArm: geometry visual mesh filename=file:///home/marguedas/.ros/nao_meshes/meshes/V40/visual/co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 scale=0.1 0.1 0.1
- link RHip: geometry visual mesh filename=file:///home/marguedas/.ros/nao_meshes/meshes/V40/visual/co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 scale=0.1 0.1 0.1
- link RPelvis: geometry visual mesh filename=file:///home/marguedas/.ros/nao_meshes/meshes/V40/visual/co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 scale=0.1 0.1 0.1
- link RShoulder: geometry visual mesh filename=file:///home/marguedas/.ros/nao_meshes/meshes/V40/visual/co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 scale=0.1 0.1 0.1
- link RThigh: geometry visual mesh filename=file:///home/marguedas/.ros/nao_meshes/meshes/V40/visual/co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 scale=0.1 0.1 0.1
- link RTibia: geometry visual mesh filename=file:///home/marguedas/.ros/nao_meshes/meshes/V40/visual/co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 scale=0.1 0.1 0.1
- link l_ankle: geometry visual mesh filename=file:///home/marguedas/.ros/nao_meshes/meshes/V40/visual/co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 scale=0.1 0.1 0.1
- link l_gripper: geometry visual mesh filename=file:///home/marguedas/.ros/nao_meshes/meshes/V40/visual/co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 scale=0.1 0.1 0.1
- link l_wrist: geometry visual mesh filename=file:///home/marguedas/.ros/nao_meshes/meshes/V40/visual/co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 scale=0.1 0.1 0.1
- link r_ankle: geometry visual mesh filename=file:///home/marguedas/.ros/nao_meshes/meshes/V40/visual/co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 scale=0.1 0.1 0.1
- link r_gripper: geometry visual mesh filename=file:///home/marguedas/.ros/nao_meshes/meshes/V40/visual/co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 scale=0.1 0.1 0.1
- link r_wrist: geometry visual mesh filename=file:///home/marguedas/.ros/nao_meshes/meshes/V40/visual/co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 scale=0.1 0.1 0.1
- link torso: geometry visual mesh filename=file:///home/marguedas/.ros/nao_meshes/meshes/V40/visual/co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 scale=0.1 0.1 0.1
