Commit message: resulting files

File: outputs/naorvizlegs.xacro (robot description, xacro)
@@ -4,6 +4,6 @@
 		<parent link="torso"/>
 		<child link="LPelvis"/>
-		<origin rpy="0 0 0" xyz="0 0 0"/>
-		<axis xyz="0 0 0"/>
+		<origin rpy="0 0 0" xyz="0 0.05 -0.085"/>
+		<axis xyz="0 0.707106 -0.707106"/>
 		<limit effort="3.2" lower="-1.14529" upper="0.740718" velocity="4.16174"/>
 	</joint>
@@ -11,11 +11,10 @@
 		<visual>
 			<geometry>
-				<mesh filename="file:///home/marguedas/.ros/nao_meshes/meshes/V40/visual/LPelvis.obj" scale="0 0 0"/>
-			</geometry>
-			<origin rpy="0 0 0" xyz="0 0 0"/>
-		</visual>
-		<collision>
-			<geometry>
-				<mesh filename="file:///home/marguedas/.ros/nao_meshes/meshes/V40/collision/LPelvis.ply" scale="0 0 0"/>
+				<mesh filename="file:///home/marguedas/.ros/nao_meshes/meshes/V40/visual/LPelvis.obj" scale="0.001 0.001 0.001"/>
+			</geometry>
+		</visual>
+		<collision>
+			<geometry>
+				<mesh filename="file:///home/marguedas/.ros/nao_meshes/meshes/V40/collision/LPelvis.ply" scale="0.001 0.001 0.001"/>
 			</geometry>
 		</collision>
@@ -23,5 +22,5 @@
 			<mass value="0.06981"/>
 			<inertia ixx="8.15023e-05" ixy="-4.99449e-06" ixz="1.27482e-05" iyy="0.000101326" iyz="2.34547e-05" izz="6.26236e-05"/>
-			<origin rpy="0 0 0" xyz="0 0 0"/>
+			<origin rpy="0 0 0" xyz="-0.00781 -0.01114 0.02661"/>
 		</inertial>
 	</link>
@@ -30,5 +29,5 @@
 		<child link="LHip"/>
 		<origin rpy="0 0 0" xyz="0 0 0"/>
-		<axis xyz="0 0 0"/>
+		<axis xyz="1.0 0 0"/>
 		<limit effort="3.2" lower="-0.379435" upper="0.79046" velocity="4.16174"/>
 	</joint>
@@ -36,11 +35,10 @@
 		<visual>
 			<geometry>
-				<mesh filename="file:///home/marguedas/.ros/nao_meshes/meshes/V40/visual/LHip.obj" scale="0 0 0"/>
-			</geometry>
-			<origin rpy="0 0 0" xyz="0 0 0"/>
-		</visual>
-		<collision>
-			<geometry>
-				<mesh filename="file:///home/marguedas/.ros/nao_meshes/meshes/V40/collision/LHip.ply" scale="0 0 0"/>
+				<mesh filename="file:///home/marguedas/.ros/nao_meshes/meshes/V40/visual/LHip.obj" scale="0.001 0.001 0.001"/>
+			</geometry>
+		</visual>
+		<collision>
+			<geometry>
+				<mesh filename="file:///home/marguedas/.ros/nao_meshes/meshes/V40/collision/LHip.ply" scale="0.001 0.001 0.001"/>
 			</geometry>
 		</collision>
@@ -48,5 +46,5 @@
 			<mass value="0.13053"/>
 			<inertia ixx="2.75835e-05" ixy="-2.233e-08" ixz="-4.08164e-06" iyy="9.82706e-05" iyz="-4.19e-09" izz="8.80997e-05"/>
-			<origin rpy="0 0 0" xyz="0 0 0"/>
+			<origin rpy="0 0 0" xyz="-0.01549 0.00029 -0.00515"/>
 		</inertial>
 	</link>
@@ -55,5 +53,5 @@
 		<child link="LThigh"/>
 		<origin rpy="0 0 0" xyz="0 0 0"/>
-		<axis xyz="0 0 0"/>
+		<axis xyz="0 1.0 0"/>
 		<limit effort="3.2" lower="-1.53589" upper="0.48398" velocity="6.40239"/>
 	</joint>
@@ -61,11 +59,10 @@
 		<visual>
 			<geometry>
-				<mesh filename="file:///home/marguedas/.ros/nao_meshes/meshes/V40/visual/LThigh.obj" scale="0 0 0"/>
-			</geometry>
-			<origin rpy="0 0 0" xyz="0 0 0"/>
-		</visual>
-		<collision>
-			<geometry>
-				<mesh filename="file:///home/marguedas/.ros/nao_meshes/meshes/V40/collision/LThigh.ply" scale="0 0 0"/>
+				<mesh filename="file:///home/marguedas/.ros/nao_meshes/meshes/V40/visual/LThigh.obj" scale="0.001 0.001 0.001"/>
+			</geometry>
+		</visual>
+		<collision>
+			<geometry>
+				<mesh filename="file:///home/marguedas/.ros/nao_meshes/meshes/V40/collision/LThigh.ply" scale="0.001 0.001 0.001"/>
 			</geometry>
 		</collision>
@@ -73,5 +70,5 @@
 			<mass value="0.38968"/>
 			<inertia ixx="0.00163672" ixy="9.2451e-07" ixz="8.53067e-05" iyy="0.00159107" iyz="3.83616e-05" izz="0.000303743"/>
-			<origin rpy="0 0 0" xyz="0 0 0"/>
+			<origin rpy="0 0 0" xyz="0.00138 0.00221 -0.05373"/>
 		</inertial>
 	</link>
@@ -79,6 +76,6 @@
 		<parent link="LThigh"/>
 		<child link="LTibia"/>
-		<origin rpy="0 0 0" xyz="0 0 0"/>
-		<axis xyz="0 0 0"/>
+		<origin rpy="0 0 0" xyz="0 0 -0.1"/>
+		<axis xyz="0 1.0 0"/>
 		<limit effort="3.2" lower="-0.0923279" upper="2.11255" velocity="6.40239"/>
 	</joint>
@@ -86,11 +83,10 @@
 		<visual>
 			<geometry>
-				<mesh filename="file:///home/marguedas/.ros/nao_meshes/meshes/V40/visual/LTibia.obj" scale="0 0 0"/>
-			</geometry>
-			<origin rpy="0 0 0" xyz="0 0 0"/>
-		</visual>
-		<collision>
-			<geometry>
-				<mesh filename="file:///home/marguedas/.ros/nao_meshes/meshes/V40/collision/LTibia.ply" scale="0 0 0"/>
+				<mesh filename="file:///home/marguedas/.ros/nao_meshes/meshes/V40/visual/LTibia.obj" scale="0.001 0.001 0.001"/>
+			</geometry>
+		</visual>
+		<collision>
+			<geometry>
+				<mesh filename="file:///home/marguedas/.ros/nao_meshes/meshes/V40/collision/LTibia.ply" scale="0.001 0.001 0.001"/>
 			</geometry>
 		</collision>
@@ -98,5 +94,5 @@
 			<mass value="0.29142"/>
 			<inertia ixx="0.00118208" ixy="6.3362e-07" ixz="3.6497e-05" iyy="0.00112865" iyz="3.94952e-05" izz="0.000193227"/>
-			<origin rpy="0 0 0" xyz="0 0 0"/>
+			<origin rpy="0 0 0" xyz="0.00453 0.00225 -0.04936"/>
 		</inertial>
 	</link>
@@ -104,6 +100,6 @@
 		<parent link="LTibia"/>
 		<child link="l_ankle"/>
-		<origin rpy="0 0 0" xyz="0 0 0"/>
-		<axis xyz="0 0 0"/>
+		<origin rpy="0 0 0" xyz="0 0 -0.1029"/>
+		<axis xyz="0 1.0 0"/>
 		<limit effort="3.2" lower="-1.18944" upper="0.922581" velocity="6.40239"/>
 	</joint>
@@ -111,11 +107,10 @@
 		<visual>
 			<geometry>
-				<mesh filename="file:///home/marguedas/.ros/nao_meshes/meshes/V40/visual/l_ankle.obj" scale="0 0 0"/>
-			</geometry>
-			<origin rpy="0 0 0" xyz="0 0 0"/>
-		</visual>
-		<collision>
-			<geometry>
-				<mesh filename="file:///home/marguedas/.ros/nao_meshes/meshes/V40/collision/l_ankle.ply" scale="0 0 0"/>
+				<mesh filename="file:///home/marguedas/.ros/nao_meshes/meshes/V40/visual/l_ankle.obj" scale="0.001 0.001 0.001"/>
+			</geometry>
+		</visual>
+		<collision>
+			<geometry>
+				<mesh filename="file:///home/marguedas/.ros/nao_meshes/meshes/V40/collision/l_ankle.ply" scale="0.001 0.001 0.001"/>
 			</geometry>
 		</collision>
@@ -123,18 +118,26 @@
 			<mass value="0.13416"/>
 			<inertia ixx="3.85098e-05" ixy="-2.634e-08" ixz="3.86194e-06" iyy="7.42653e-05" iyz="1.834e-08" izz="5.48654e-05"/>
-			<origin rpy="0 0 0" xyz="0 0 0"/>
-		</inertial>
-	</link>
-	<joint name="l_sole_joint" type="fixed">
+			<origin rpy="0 0 0" xyz="0.00045 0.00029 0.00685"/>
+		</inertial>
+	</link>
+	<joint name="LAnkleRoll" type="revolute">
 		<parent link="l_ankle"/>
-		<child link="l_sole"/>
-		<origin rpy="0 0 0" xyz="0 0 0"/>
-	</joint>
-	<link name="l_sole"/>
+		<child link="LFeet"/>
+		<origin rpy="0 0 0" xyz="0 0 0"/>
+		<axis xyz="1.0 0 0"/>
+		<limit effort="3.2" lower="-0.397761" upper="0.768992" velocity="4.16174"/>
+	</joint>
+	<link name="LFeet">
+		<inertial>
+			<mass value="0.16184"/>
+			<inertia ixx="0.000269442" ixy="-5.69572e-06" ixz="0.000139379" iyy="0.000644343" iyz="1.87409e-05" izz="0.000525757"/>
+			<origin rpy="0 0 0" xyz="0.02542 0.0033 -0.03239"/>
+		</inertial>
+	</link>
 	<joint name="RHipYawPitch" type="revolute">
 		<parent link="torso"/>
 		<child link="RPelvis"/>
-		<origin rpy="0 0 0" xyz="0 0 0"/>
-		<axis xyz="0 0 0"/>
+		<origin rpy="0 0 0" xyz="0 -0.05 -0.085"/>
+		<axis xyz="0 0.707106 0.707106"/>
 		<limit effort="3.2" lower="-1.14529" upper="0.740718" velocity="4.16174"/>
 	</joint>
@@ -142,11 +145,10 @@
 		<visual>
 			<geometry>
-				<mesh filename="file:///home/marguedas/.ros/nao_meshes/meshes/V40/visual/RPelvis.obj" scale="0 0 0"/>
-			</geometry>
-			<origin rpy="0 0 0" xyz="0 0 0"/>
-		</visual>
-		<collision>
-			<geometry>
-				<mesh filename="file:///home/marguedas/.ros/nao_meshes/meshes/V40/collision/RPelvis.ply" scale="0 0 0"/>
+				<mesh filename="file:///home/marguedas/.ros/nao_meshes/meshes/V40/visual/RPelvis.obj" scale="0.001 0.001 0.001"/>
+			</geometry>
+		</visual>
+		<collision>
+			<geometry>
+				<mesh filename="file:///home/marguedas/.ros/nao_meshes/meshes/V40/collision/RPelvis.ply" scale="0.001 0.001 0.001"/>
 			</geometry>
 		</collision>
@@ -154,5 +156,5 @@
 			<mass value="0.06981"/>
 			<inertia ixx="8.9972e-05" ixy="5.00219e-06" ixz="1.27352e-05" iyy="0.000105526" iyz="-2.77008e-05" izz="6.68872e-05"/>
-			<origin rpy="0 0 0" xyz="0 0 0"/>
+			<origin rpy="0 0 0" xyz="-0.00781 0.01114 0.02661"/>
 		</inertial>
 	</link>
@@ -161,5 +163,5 @@
 		<child link="RHip"/>
 		<origin rpy="0 0 0" xyz="0 0 0"/>
-		<axis xyz="0 0 0"/>
+		<axis xyz="1.0 0 0"/>
 		<limit effort="3.2" lower="-0.79046" upper="0.379435" velocity="4.16174"/>
 	</joint>
@@ -167,11 +169,10 @@
 		<visual>
 			<geometry>
-				<mesh filename="file:///home/marguedas/.ros/nao_meshes/meshes/V40/visual/RHip.obj" scale="0 0 0"/>
-			</geometry>
-			<origin rpy="0 0 0" xyz="0 0 0"/>
-		</visual>
-		<collision>
-			<geometry>
-				<mesh filename="file:///home/marguedas/.ros/nao_meshes/meshes/V40/collision/RHip.ply" scale="0 0 0"/>
+				<mesh filename="file:///home/marguedas/.ros/nao_meshes/meshes/V40/visual/RHip.obj" scale="0.001 0.001 0.001"/>
+			</geometry>
+		</visual>
+		<collision>
+			<geometry>
+				<mesh filename="file:///home/marguedas/.ros/nao_meshes/meshes/V40/collision/RHip.ply" scale="0.001 0.001 0.001"/>
 			</geometry>
 		</collision>
@@ -179,5 +180,5 @@
 			<mass value="0.13053"/>
 			<inertia ixx="2.75865e-05" ixy="-1.919e-08" ixz="-4.10822e-06" iyy="9.827e-05" iyz="2.51e-09" izz="8.81033e-05"/>
-			<origin rpy="0 0 0" xyz="0 0 0"/>
+			<origin rpy="0 0 0" xyz="-0.01549 -0.00029 -0.00515"/>
 		</inertial>
 	</link>
@@ -186,5 +187,5 @@
 		<child link="RThigh"/>
 		<origin rpy="0 0 0" xyz="0 0 0"/>
-		<axis xyz="0 0 0"/>
+		<axis xyz="0 1.0 0"/>
 		<limit effort="3.2" lower="-1.53589" upper="0.48398" velocity="6.40239"/>
 	</joint>
@@ -192,11 +193,10 @@
 		<visual>
 			<geometry>
-				<mesh filename="file:///home/marguedas/.ros/nao_meshes/meshes/V40/visual/RThigh.obj" scale="0 0 0"/>
-			</geometry>
-			<origin rpy="0 0 0" xyz="0 0 0"/>
-		</visual>
-		<collision>
-			<geometry>
-				<mesh filename="file:///home/marguedas/.ros/nao_meshes/meshes/V40/collision/RThigh.ply" scale="0 0 0"/>
+				<mesh filename="file:///home/marguedas/.ros/nao_meshes/meshes/V40/visual/RThigh.obj" scale="0.001 0.001 0.001"/>
+			</geometry>
+		</visual>
+		<collision>
+			<geometry>
+				<mesh filename="file:///home/marguedas/.ros/nao_meshes/meshes/V40/collision/RThigh.ply" scale="0.001 0.001 0.001"/>
 			</geometry>
 		</collision>
@@ -204,5 +204,5 @@
 			<mass value="0.38968"/>
 			<inertia ixx="0.00163748" ixy="-8.3954e-07" ixz="8.5883e-05" iyy="0.00159221" iyz="-3.91763e-05" izz="0.000303978"/>
-			<origin rpy="0 0 0" xyz="0 0 0"/>
+			<origin rpy="0 0 0" xyz="0.00138 -0.00221 -0.05373"/>
 		</inertial>
 	</link>
@@ -210,6 +210,6 @@
 		<parent link="RThigh"/>
 		<child link="RTibia"/>
-		<origin rpy="0 0 0" xyz="0 0 0"/>
-		<axis xyz="0 0 0"/>
+		<origin rpy="0 0 0" xyz="0 0 -0.1"/>
+		<axis xyz="0 1.0 0"/>
 		<limit effort="3.2" lower="-0.0923279" upper="2.11255" velocity="6.40239"/>
 	</joint>
@@ -217,11 +217,10 @@
 		<visual>
 			<geometry>
-				<mesh filename="file:///home/marguedas/.ros/nao_meshes/meshes/V40/visual/RTibia.obj" scale="0 0 0"/>
-			</geometry>
-			<origin rpy="0 0 0" xyz="0 0 0"/>
-		</visual>
-		<collision>
-			<geometry>
-				<mesh filename="file:///home/marguedas/.ros/nao_meshes/meshes/V40/collision/RTibia.ply" scale="0 0 0"/>
+				<mesh filename="file:///home/marguedas/.ros/nao_meshes/meshes/V40/visual/RTibia.obj" scale="0.001 0.001 0.001"/>
+			</geometry>
+		</visual>
+		<collision>
+			<geometry>
+				<mesh filename="file:///home/marguedas/.ros/nao_meshes/meshes/V40/collision/RTibia.ply" scale="0.001 0.001 0.001"/>
 			</geometry>
 		</collision>
@@ -229,5 +228,5 @@
 			<mass value="0.29142"/>
 			<inertia ixx="0.00118283" ixy="-8.965e-07" ixz="2.79969e-05" iyy="0.00112828" iyz="-3.8476e-05" izz="0.000191453"/>
-			<origin rpy="0 0 0" xyz="0 0 0"/>
+			<origin rpy="0 0 0" xyz="0.00453 -0.00225 -0.04936"/>
 		</inertial>
 	</link>
@@ -235,6 +234,6 @@
 		<parent link="RTibia"/>
 		<child link="r_ankle"/>
-		<origin rpy="0 0 0" xyz="0 0 0"/>
-		<axis xyz="0 0 0"/>
+		<origin rpy="0 0 0" xyz="0 0 -0.1029"/>
+		<axis xyz="0 1.0 0"/>
 		<limit effort="3.2" lower="-1.1863" upper="0.932006" velocity="6.40239"/>
 	</joint>
@@ -242,11 +241,10 @@
 		<visual>
 			<geometry>
-				<mesh filename="file:///home/marguedas/.ros/nao_meshes/meshes/V40/visual/r_ankle.obj" scale="0 0 0"/>
-			</geometry>
-			<origin rpy="0 0 0" xyz="0 0 0"/>
-		</visual>
-		<collision>
-			<geometry>
-				<mesh filename="file:///home/marguedas/.ros/nao_meshes/meshes/V40/collision/r_ankle.ply" scale="0 0 0"/>
+				<mesh filename="file:///home/marguedas/.ros/nao_meshes/meshes/V40/visual/r_ankle.obj" scale="0.001 0.001 0.001"/>
+			</geometry>
+		</visual>
+		<collision>
+			<geometry>
+				<mesh filename="file:///home/marguedas/.ros/nao_meshes/meshes/V40/collision/r_ankle.ply" scale="0.001 0.001 0.001"/>
 			</geometry>
 		</collision>
@@ -254,12 +252,20 @@
 			<mass value="0.13416"/>
 			<inertia ixx="3.85081e-05" ixy="6.434e-08" ixz="3.87466e-06" iyy="7.43108e-05" iyz="-4.58e-09" izz="5.49131e-05"/>
-			<origin rpy="0 0 0" xyz="0 0 0"/>
-		</inertial>
-	</link>
-	<joint name="r_sole_joint" type="fixed">
+			<origin rpy="0 0 0" xyz="0.00045 -0.00029 0.00685"/>
+		</inertial>
+	</link>
+	<joint name="RAnkleRoll" type="revolute">
 		<parent link="r_ankle"/>
-		<child link="r_sole"/>
-		<origin rpy="0 0 0" xyz="0 0 0"/>
-	</joint>
-	<link name="r_sole"/>
+		<child link="RFeet"/>
+		<origin rpy="0 0 0" xyz="0 0 0"/>
+		<axis xyz="1.0 0 0"/>
+		<limit effort="3.2" lower="-0.768992" upper="0.397935" velocity="4.16174"/>
+	</joint>
+	<link name="RFeet">
+		<inertial>
+			<mass value="0.16184"/>
+			<inertia ixx="0.000269302" ixy="5.87505e-06" ixz="0.000139133" iyy="0.000643474" iyz="-1.88492e-05" izz="0.000525035"/>
+			<origin rpy="0 0 0" xyz="0.02542 -0.0033 -0.03239"/>
+		</inertial>
+	</link>
 </robot>
