Commit message: remove colors in gazebo tags

File: outputs/naogazeboGazebo.xacro (robot description, xacro)
@@ -2,5 +2,5 @@
 <robot xmlns:xacro="http://www.ros.org/wiki/xacro">
 	<gazebo reference="LThigh">
-		<material>Gazebo/Red</material>
+		<material>Gazebo/White</material>
 		<turnGravityOff>false</turnGravityOff>
 		<mu1>0.5</mu1>
@@ -9,5 +9,5 @@
 	</gazebo>
 	<gazebo reference="l_wrist">
-		<material>Gazebo/Red</material>
+		<material>Gazebo/White</material>
 		<turnGravityOff>false</turnGravityOff>
 		<mu1>0.5</mu1>
@@ -16,5 +16,5 @@
 	</gazebo>
 	<gazebo reference="RBicep">
-		<material>Gazebo/Blue</material>
+		<material>Gazebo/White</material>
 		<turnGravityOff>false</turnGravityOff>
 		<mu1>0.5</mu1>
@@ -23,5 +23,5 @@
 	</gazebo>
 	<gazebo reference="l_gripper">
-		<material>Gazebo/Red</material>
+		<material>Gazebo/White</material>
 		<turnGravityOff>false</turnGravityOff>
 		<mu1>0.5</mu1>
@@ -30,5 +30,5 @@
 	</gazebo>
 	<gazebo reference="r_sole">
-		<material>Gazebo/Orange</material>
+		<material>Gazebo/White</material>
 		<turnGravityOff>false</turnGravityOff>
 		<mu1>0.5</mu1>
@@ -37,5 +37,5 @@
 	</gazebo>
 	<gazebo reference="RFeet">
-		<material>Gazebo/Blue</material>
+		<material>Gazebo/White</material>
 		<turnGravityOff>false</turnGravityOff>
 		<mu1>0.5</mu1>
@@ -51,5 +51,5 @@
 	</gazebo>
 	<gazebo reference="RThigh">
-		<material>Gazebo/Blue</material>
+		<material>Gazebo/White</material>
 		<turnGravityOff>false</turnGravityOff>
 		<mu1>0.5</mu1>
@@ -58,5 +58,5 @@
 	</gazebo>
 	<gazebo reference="r_ankle">
-		<material>Gazebo/Blue</material>
+		<material>Gazebo/White</material>
 		<turnGravityOff>false</turnGravityOff>
 		<mu1>0.5</mu1>
@@ -72,5 +72,5 @@
 	</gazebo>
 	<gazebo reference="LTibia">
-		<material>Gazebo/Red</material>
+		<material>Gazebo/White</material>
 		<turnGravityOff>false</turnGravityOff>
 		<mu1>0.5</mu1>
@@ -79,5 +79,5 @@
 	</gazebo>
 	<gazebo reference="r_wrist">
-		<material>Gazebo/Blue</material>
+		<material>Gazebo/White</material>
 		<turnGravityOff>false</turnGravityOff>
 		<mu1>0.5</mu1>
@@ -93,5 +93,5 @@
 	</gazebo>
 	<gazebo reference="LElbow">
-		<material>Gazebo/Red</material>
+		<material>Gazebo/White</material>
 		<turnGravityOff>false</turnGravityOff>
 		<mu1>0.5</mu1>
@@ -100,5 +100,5 @@
 	</gazebo>
 	<gazebo reference="RElbow">
-		<material>Gazebo/Blue</material>
+		<material>Gazebo/White</material>
 		<turnGravityOff>false</turnGravityOff>
 		<mu1>0.5</mu1>
@@ -107,5 +107,5 @@
 	</gazebo>
 	<gazebo reference="l_ankle">
-		<material>Gazebo/Red</material>
+		<material>Gazebo/White</material>
 		<turnGravityOff>false</turnGravityOff>
 		<mu1>0.5</mu1>
@@ -121,5 +121,5 @@
 	</gazebo>
 	<gazebo reference="l_sole">
-		<material>Gazebo/Orange</material>
+		<material>Gazebo/White</material>
 		<turnGravityOff>false</turnGravityOff>
 		<mu1>0.5</mu1>
@@ -128,5 +128,5 @@
 	</gazebo>
 	<gazebo reference="LForeArm">
-		<material>Gazebo/Red</material>
+		<material>Gazebo/White</material>
 		<turnGravityOff>false</turnGravityOff>
 		<mu1>0.5</mu1>
@@ -135,5 +135,5 @@
 	</gazebo>
 	<gazebo reference="RHip">
-		<material>Gazebo/Blue</material>
+		<material>Gazebo/White</material>
 		<turnGravityOff>false</turnGravityOff>
 		<mu1>0.5</mu1>
@@ -142,5 +142,5 @@
 	</gazebo>
 	<gazebo reference="RForeArm">
-		<material>Gazebo/Blue</material>
+		<material>Gazebo/White</material>
 		<turnGravityOff>false</turnGravityOff>
 		<mu1>0.5</mu1>
@@ -149,5 +149,5 @@
 	</gazebo>
 	<gazebo reference="r_gripper">
-		<material>Gazebo/Blue</material>
+		<material>Gazebo/White</material>
 		<turnGravityOff>false</turnGravityOff>
 		<mu1>0.5</mu1>
@@ -156,5 +156,5 @@
 	</gazebo>
 	<gazebo reference="LBicep">
-		<material>Gazebo/Red</material>
+		<material>Gazebo/White</material>
 		<turnGravityOff>false</turnGravityOff>
 		<mu1>0.5</mu1>
@@ -163,5 +163,5 @@
 	</gazebo>
 	<gazebo reference="RPelvis">
-		<material>Gazebo/Blue</material>
+		<material>Gazebo/White</material>
 		<turnGravityOff>false</turnGravityOff>
 		<mu1>0.5</mu1>
@@ -170,5 +170,5 @@
 	</gazebo>
 	<gazebo reference="LShoulder">
-		<material>Gazebo/Red</material>
+		<material>Gazebo/White</material>
 		<turnGravityOff>false</turnGravityOff>
 		<mu1>0.5</mu1>
@@ -177,5 +177,5 @@
 	</gazebo>
 	<gazebo reference="RTibia">
-		<material>Gazebo/Blue</material>
+		<material>Gazebo/White</material>
 		<turnGravityOff>false</turnGravityOff>
 		<mu1>0.5</mu1>
@@ -184,5 +184,5 @@
 	</gazebo>
 	<gazebo reference="RShoulder">
-		<material>Gazebo/Blue</material>
+		<material>Gazebo/White</material>
 		<turnGravityOff>false</turnGravityOff>
 		<mu1>0.5</mu1>
@@ -191,5 +191,5 @@
 	</gazebo>
 	<gazebo reference="LHip">
-		<material>Gazebo/Red</material>
+		<material>Gazebo/White</material>
 		<turnGravityOff>false</turnGravityOff>
 		<mu1>0.5</mu1>
@@ -198,5 +198,5 @@
 	</gazebo>
 	<gazebo reference="LPelvis">
-		<material>Gazebo/Red</material>
+		<material>Gazebo/White</material>
 		<turnGravityOff>false</turnGravityOff>
 		<mu1>0.5</mu1>
@@ -205,5 +205,5 @@
 	</gazebo>
 	<gazebo reference="LFeet">
-		<material>Gazebo/Red</material>
+		<material>Gazebo/White</material>
 		<turnGravityOff>false</turnGravityOff>
 		<mu1>0.5</mu1>
