Commit message: added gazebo tag parsing in gazeboUrdf.py

File: outputs/naoOut.urdf (robot description, URDF)
Before this commit: robot naoH25V40, 30 links, 29 joints
Links:
- link Head: geometry collision mesh filename=package://nao_meshes/meshes/V40/visual/collada/Head.dae scale=0.1 0.1 0.1; visual mesh filename=package://nao_meshes/meshes/V40/visual/collada/Head.dae scale=0.1 0.1 0.1
- link LBicep: geometry collision mesh filename=package://nao_meshes/meshes/V40/visual/collada/LBicep.dae scale=0.1 0.1 0.1; visual mesh filename=package://nao_meshes/meshes/V40/visual/collada/LBicep.dae scale=0.1 0.1 0.1
- link LFeet: geometry collision mesh filename=package://nao_meshes/meshes/V40/visual/collada/LFeet.dae scale=0.1 0.1 0.1; visual mesh filename=package://nao_meshes/meshes/V40/visual/collada/LFeet.dae scale=0.1 0.1 0.1
- link LForeArm: geometry collision mesh filename=package://nao_meshes/meshes/V40/visual/collada/LForeArm.dae scale=0.1 0.1 0.1; visual mesh filename=package://nao_meshes/meshes/V40/visual/collada/LForeArm.dae scale=0.1 0.1 0.1
- link LHip: geometry collision mesh filename=package://nao_meshes/meshes/V40/visual/collada/LHip.dae scale=0.1 0.1 0.1; visual mesh filename=package://nao_meshes/meshes/V40/visual/collada/LHip.dae scale=0.1 0.1 0.1
- link LPelvis: geometry collision mesh filename=package://nao_meshes/meshes/V40/visual/collada/LPelvis.dae scale=0.1 0.1 0.1; visual mesh filename=package://nao_meshes/meshes/V40/visual/collada/LPelvis.dae scale=0.1 0.1 0.1
- link LShoulder: geometry collision mesh filename=package://nao_meshes/meshes/V40/visual/collada/LShoulder.dae scale=0.1 0.1 0.1; visual mesh filename=package://nao_meshes/meshes/V40/visual/collada/LShoulder.dae scale=0.1 0.1 0.1
- link LThigh: geometry collision mesh filename=package://nao_meshes/meshes/V40/visual/collada/LThigh.dae scale=0.1 0.1 0.1; visual mesh filename=package://nao_meshes/meshes/V40/visual/collada/LThigh.dae scale=0.1 0.1 0.1
- link LTibia: geometry collision mesh filename=package://nao_meshes/meshes/V40/visual/collada/LTibia.dae scale=0.1 0.1 0.1; visual mesh filename=package://nao_meshes/meshes/V40/visual/collada/LTibia.dae scale=0.1 0.1 0.1
- link Neck: geometry collision mesh filename=package://nao_meshes/meshes/V40/visual/collada/Neck.dae scale=0.1 0.1 0.1; visual mesh filename=package://nao_meshes/meshes/V40/visual/collada/Neck.dae scale=0.1 0.1 0.1
- link RBicep: geometry collision mesh filename=package://nao_meshes/meshes/V40/visual/collada/RBicep.dae scale=0.1 0.1 0.1; visual mesh filename=package://nao_meshes/meshes/V40/visual/collada/RBicep.dae scale=0.1 0.1 0.1
- link RFeet: geometry collision mesh filename=package://nao_meshes/meshes/V40/visual/collada/RFeet.dae scale=0.1 0.1 0.1; visual mesh filename=package://nao_meshes/meshes/V40/visual/collada/RFeet.dae scale=0.1 0.1 0.1
- link RForeArm: geometry collision mesh filename=package://nao_meshes/meshes/V40/visual/collada/RForeArm.dae scale=0.1 0.1 0.1; visual mesh filename=package://nao_meshes/meshes/V40/visual/collada/RForeArm.dae scale=0.1 0.1 0.1
- link RHip: geometry collision mesh filename=package://nao_meshes/meshes/V40/visual/collada/RHip.dae scale=0.1 0.1 0.1; visual mesh filename=package://nao_meshes/meshes/V40/visual/collada/RHip.dae scale=0.1 0.1 0.1
- link RPelvis: geometry collision mesh filename=package://nao_meshes/meshes/V40/visual/collada/RPelvis.dae scale=0.1 0.1 0.1; visual mesh filename=package://nao_meshes/meshes/V40/visual/collada/RPelvis.dae scale=0.1 0.1 0.1
- link RShoulder: geometry collision mesh filename=package://nao_meshes/meshes/V40/visual/collada/RShoulder.dae scale=0.1 0.1 0.1; visual mesh filename=package://nao_meshes/meshes/V40/visual/collada/RShoulder.dae scale=0.1 0.1 0.1
- link RThigh: geometry collision mesh filename=package://nao_meshes/meshes/V40/visual/collada/RThigh.dae scale=0.1 0.1 0.1; visual mesh filename=package://nao_meshes/meshes/V40/visual/collada/RThigh.dae scale=0.1 0.1 0.1
- link RTibia: geometry collision mesh filename=package://nao_meshes/meshes/V40/visual/collada/RTibia.dae scale=0.1 0.1 0.1; visual mesh filename=package://nao_meshes/meshes/V40/visual/collada/RTibia.dae scale=0.1 0.1 0.1
- link l_ankle: geometry collision mesh filename=package://nao_meshes/meshes/V40/visual/collada/l_ankle.dae scale=0.1 0.1 0.1; visual mesh filename=package://nao_meshes/meshes/V40/visual/collada/l_ankle.dae scale=0.1 0.1 0.1
- link l_gripper: geometry collision mesh filename=package://nao_meshes/meshes/V40/visual/collada/l_gripper.dae scale=0.1 0.1 0.1; visual mesh filename=package://nao_meshes/meshes/V40/visual/collada/l_gripper.dae scale=0.1 0.1 0.1
- link l_wrist: geometry collision mesh filename=package://nao_meshes/meshes/V40/visual/collada/l_wrist.dae scale=0.1 0.1 0.1; visual mesh filename=package://nao_meshes/meshes/V40/visual/collada/l_wrist.dae scale=0.1 0.1 0.1
- link r_ankle: geometry collision mesh filename=package://nao_meshes/meshes/V40/visual/collada/r_ankle.dae scale=0.1 0.1 0.1; visual mesh filename=package://nao_meshes/meshes/V40/visual/collada/r_ankle.dae scale=0.1 0.1 0.1
- link r_gripper: geometry collision mesh filename=package://nao_meshes/meshes/V40/visual/collada/r_gripper.dae scale=0.1 0.1 0.1; visual mesh filename=package://nao_meshes/meshes/V40/visual/collada/r_gripper.dae scale=0.1 0.1 0.1
- link r_wrist: geometry collision mesh filename=package://nao_meshes/meshes/V40/visual/collada/r_wrist.dae scale=0.1 0.1 0.1; visual mesh filename=package://nao_meshes/meshes/V40/visual/collada/r_wrist.dae scale=0.1 0.1 0.1
- link torso: geometry collision mesh filename=package://nao_meshes/meshes/V40/visual/collada/torso.dae scale=0.1 0.1 0.1; visual mesh filename=package://nao_meshes/meshes/V40/visual/collada/torso.dae scale=0.1 0.1 0.1

File: outputs/naoOutGazebo.xacro (robot description, xacro)
@@ -1,4 +1,16 @@
 <?xml version="1.0" ?>
 <robot xmlns:xacro="http://www.ros.org/wiki/xacro">
+	<gazebo>
+		<plugin filename="libgazebo_ros_control.so" name="gazebo_ros_control">
+			<robotNamespace>/nao_dcm</robotNamespace>
+			<robotSimType>gazebo_ros_control/DefaultRobotHWSim</robotSimType>
+		</plugin>
+		<plugin filename="libroboticsgroup_gazebo_mimic_joint_plugin.so" name="mimic_hipyawpitch">
+			<joint>LHipYawPitch</joint>
+			<mimicjoint>RHipYawPitch</mimicjoint>
+			<multiplier>1.0</multiplier>
+			<offset>0.0</offset>
+		</plugin>
+	</gazebo>
 	<gazebo reference="LThigh">
 		<material>Gazebo/White</material>

File: outputs/naoOutarms.xacro (robot description, xacro)
@@ -11,10 +11,10 @@
 		<visual>
 			<geometry>
-				<mesh filename="file:///home/marguedas/.ros/nao_meshes/meshes/V40/visual/collada/LShoulder.dae" scale="0.1 0.1 0.1"/>
-			</geometry>
-		</visual>
-		<collision>
-			<geometry>
-				<mesh filename="file:///home/marguedas/.ros/nao_meshes/meshes/V40/visual/collada/LShoulder.dae" scale="0.1 0.1 0.1"/>
+				<mesh filename="package://nao_meshes/meshes/V40/visual/collada/LShoulder.dae" scale="0.1 0.1 0.1"/>
+			</geometry>
+		</visual>
+		<collision>
+			<geometry>
+				<mesh filename="package://nao_meshes/meshes/V40/visual/collada/LShoulder.dae" scale="0.1 0.1 0.1"/>
 			</geometry>
 		</collision>
@@ -35,10 +35,10 @@
 		<visual>
 			<geometry>
-				<mesh filename="file:///home/marguedas/.ros/nao_meshes/meshes/V40/visual/collada/LBicep.dae" scale="0.1 0.1 0.1"/>
-			</geometry>
-		</visual>
-		<collision>
-			<geometry>
-				<mesh filename="file:///home/marguedas/.ros/nao_meshes/meshes/V40/visual/collada/LBicep.dae" scale="0.1 0.1 0.1"/>
+				<mesh filename="package://nao_meshes/meshes/V40/visual/collada/LBicep.dae" scale="0.1 0.1 0.1"/>
+			</geometry>
+		</visual>
+		<collision>
+			<geometry>
+				<mesh filename="package://nao_meshes/meshes/V40/visual/collada/LBicep.dae" scale="0.1 0.1 0.1"/>
 			</geometry>
 		</collision>
@@ -73,10 +73,10 @@
 		<visual>
 			<geometry>
-				<mesh filename="file:///home/marguedas/.ros/nao_meshes/meshes/V40/visual/collada/LForeArm.dae" scale="0.1 0.1 0.1"/>
-			</geometry>
-		</visual>
-		<collision>
-			<geometry>
-				<mesh filename="file:///home/marguedas/.ros/nao_meshes/meshes/V40/visual/collada/LForeArm.dae" scale="0.1 0.1 0.1"/>
+				<mesh filename="package://nao_meshes/meshes/V40/visual/collada/LForeArm.dae" scale="0.1 0.1 0.1"/>
+			</geometry>
+		</visual>
+		<collision>
+			<geometry>
+				<mesh filename="package://nao_meshes/meshes/V40/visual/collada/LForeArm.dae" scale="0.1 0.1 0.1"/>
 			</geometry>
 		</collision>
@@ -97,10 +97,10 @@
 		<visual>
 			<geometry>
-				<mesh filename="file:///home/marguedas/.ros/nao_meshes/meshes/V40/visual/collada/l_wrist.dae" scale="0.1 0.1 0.1"/>
-			</geometry>
-		</visual>
-		<collision>
-			<geometry>
-				<mesh filename="file:///home/marguedas/.ros/nao_meshes/meshes/V40/visual/collada/l_wrist.dae" scale="0.1 0.1 0.1"/>
+				<mesh filename="package://nao_meshes/meshes/V40/visual/collada/l_wrist.dae" scale="0.1 0.1 0.1"/>
+			</geometry>
+		</visual>
+		<collision>
+			<geometry>
+				<mesh filename="package://nao_meshes/meshes/V40/visual/collada/l_wrist.dae" scale="0.1 0.1 0.1"/>
 			</geometry>
 		</collision>
@@ -119,10 +119,10 @@
 		<visual>
 			<geometry>
-				<mesh filename="file:///home/marguedas/.ros/nao_meshes/meshes/V40/visual/collada/l_gripper.dae" scale="0.1 0.1 0.1"/>
-			</geometry>
-		</visual>
-		<collision>
-			<geometry>
-				<mesh filename="file:///home/marguedas/.ros/nao_meshes/meshes/V40/visual/collada/l_gripper.dae" scale="0.1 0.1 0.1"/>
+				<mesh filename="package://nao_meshes/meshes/V40/visual/collada/l_gripper.dae" scale="0.1 0.1 0.1"/>
+			</geometry>
+		</visual>
+		<collision>
+			<geometry>
+				<mesh filename="package://nao_meshes/meshes/V40/visual/collada/l_gripper.dae" scale="0.1 0.1 0.1"/>
 			</geometry>
 		</collision>
@@ -138,10 +138,10 @@
 		<visual>
 			<geometry>
-				<mesh filename="file:///home/marguedas/.ros/nao_meshes/meshes/V40/visual/collada/RShoulder.dae" scale="0.1 0.1 0.1"/>
-			</geometry>
-		</visual>
-		<collision>
-			<geometry>
-				<mesh filename="file:///home/marguedas/.ros/nao_meshes/meshes/V40/visual/collada/RShoulder.dae" scale="0.1 0.1 0.1"/>
+				<mesh filename="package://nao_meshes/meshes/V40/visual/collada/RShoulder.dae" scale="0.1 0.1 0.1"/>
+			</geometry>
+		</visual>
+		<collision>
+			<geometry>
+				<mesh filename="package://nao_meshes/meshes/V40/visual/collada/RShoulder.dae" scale="0.1 0.1 0.1"/>
 			</geometry>
 		</collision>
@@ -162,10 +162,10 @@
 		<visual>
 			<geometry>
-				<mesh filename="file:///home/marguedas/.ros/nao_meshes/meshes/V40/visual/collada/RBicep.dae" scale="0.1 0.1 0.1"/>
-			</geometry>
-		</visual>
-		<collision>
-			<geometry>
-				<mesh filename="file:///home/marguedas/.ros/nao_meshes/meshes/V40/visual/collada/RBicep.dae" scale="0.1 0.1 0.1"/>
+				<mesh filename="package://nao_meshes/meshes/V40/visual/collada/RBicep.dae" scale="0.1 0.1 0.1"/>
+			</geometry>
+		</visual>
+		<collision>
+			<geometry>
+				<mesh filename="package://nao_meshes/meshes/V40/visual/collada/RBicep.dae" scale="0.1 0.1 0.1"/>
 			</geometry>
 		</collision>
@@ -200,10 +200,10 @@
 		<visual>
 			<geometry>
-				<mesh filename="file:///home/marguedas/.ros/nao_meshes/meshes/V40/visual/collada/RForeArm.dae" scale="0.1 0.1 0.1"/>
-			</geometry>
-		</visual>
-		<collision>
-			<geometry>
-				<mesh filename="file:///home/marguedas/.ros/nao_meshes/meshes/V40/visual/collada/RForeArm.dae" scale="0.1 0.1 0.1"/>
+				<mesh filename="package://nao_meshes/meshes/V40/visual/collada/RForeArm.dae" scale="0.1 0.1 0.1"/>
+			</geometry>
+		</visual>
+		<collision>
+			<geometry>
+				<mesh filename="package://nao_meshes/meshes/V40/visual/collada/RForeArm.dae" scale="0.1 0.1 0.1"/>
 			</geometry>
 		</collision>
@@ -224,10 +224,10 @@
 		<visual>
 			<geometry>
-				<mesh filename="file:///home/marguedas/.ros/nao_meshes/meshes/V40/visual/collada/r_wrist.dae" scale="0.1 0.1 0.1"/>
-			</geometry>
-		</visual>
-		<collision>
-			<geometry>
-				<mesh filename="file:///home/marguedas/.ros/nao_meshes/meshes/V40/visual/collada/r_wrist.dae" scale="0.1 0.1 0.1"/>
+				<mesh filename="package://nao_meshes/meshes/V40/visual/collada/r_wrist.dae" scale="0.1 0.1 0.1"/>
+			</geometry>
+		</visual>
+		<collision>
+			<geometry>
+				<mesh filename="package://nao_meshes/meshes/V40/visual/collada/r_wrist.dae" scale="0.1 0.1 0.1"/>
 			</geometry>
 		</collision>
@@ -246,10 +246,10 @@
 		<visual>
 			<geometry>
-				<mesh filename="file:///home/marguedas/.ros/nao_meshes/meshes/V40/visual/collada/r_gripper.dae" scale="0.1 0.1 0.1"/>
-			</geometry>
-		</visual>
-		<collision>
-			<geometry>
-				<mesh filename="file:///home/marguedas/.ros/nao_meshes/meshes/V40/visual/collada/r_gripper.dae" scale="0.1 0.1 0.1"/>
+				<mesh filename="package://nao_meshes/meshes/V40/visual/collada/r_gripper.dae" scale="0.1 0.1 0.1"/>
+			</geometry>
+		</visual>
+		<collision>
+			<geometry>
+				<mesh filename="package://nao_meshes/meshes/V40/visual/collada/r_gripper.dae" scale="0.1 0.1 0.1"/>
 			</geometry>
 		</collision>

File: outputs/naoOuthead.xacro (robot description, xacro)
@@ -11,10 +11,10 @@
 		<visual>
 			<geometry>
-				<mesh filename="file:///home/marguedas/.ros/nao_meshes/meshes/V40/visual/collada/Neck.dae" scale="0.1 0.1 0.1"/>
+				<mesh filename="package://nao_meshes/meshes/V40/visual/collada/Neck.dae" scale="0.1 0.1 0.1"/>
 			</geometry>
 		</visual>
 		<collision>
 			<geometry>
-				<mesh filename="file:///home/marguedas/.ros/nao_meshes/meshes/V40/visual/collada/Neck.dae" scale="0.1 0.1 0.1"/>
+				<mesh filename="package://nao_meshes/meshes/V40/visual/collada/Neck.dae" scale="0.1 0.1 0.1"/>
 			</geometry>
 		</collision>
@@ -35,10 +35,10 @@
 		<visual>
 			<geometry>
-				<mesh filename="file:///home/marguedas/.ros/nao_meshes/meshes/V40/visual/collada/Head.dae" scale="0.1 0.1 0.1"/>
+				<mesh filename="package://nao_meshes/meshes/V40/visual/collada/Head.dae" scale="0.1 0.1 0.1"/>
 			</geometry>
 		</visual>
 		<collision>
 			<geometry>
-				<mesh filename="file:///home/marguedas/.ros/nao_meshes/meshes/V40/visual/collada/Head.dae" scale="0.1 0.1 0.1"/>
+				<mesh filename="package://nao_meshes/meshes/V40/visual/collada/Head.dae" scale="0.1 0.1 0.1"/>
 			</geometry>
 		</collision>

File: outputs/naoOutlegs.xacro (robot description, xacro)
@@ -11,10 +11,10 @@
 		<visual>
 			<geometry>
-				<mesh filename="file:///home/marguedas/.ros/nao_meshes/meshes/V40/visual/LPelvis.obj" scale="0.001 0.001 0.001"/>
-			</geometry>
-		</visual>
-		<collision>
-			<geometry>
-				<mesh filename="file:///home/marguedas/.ros/nao_meshes/meshes/V40/collision/LPelvis.ply" scale="0.001 0.001 0.001"/>
+				<mesh filename="package://nao_meshes/meshes/V40/visual/collada/LPelvis.dae" scale="0.1 0.1 0.1"/>
+			</geometry>
+		</visual>
+		<collision>
+			<geometry>
+				<mesh filename="package://nao_meshes/meshes/V40/visual/collada/LPelvis.dae" scale="0.1 0.1 0.1"/>
 			</geometry>
 		</collision>
@@ -35,10 +35,10 @@
 		<visual>
 			<geometry>
-				<mesh filename="file:///home/marguedas/.ros/nao_meshes/meshes/V40/visual/LHip.obj" scale="0.001 0.001 0.001"/>
-			</geometry>
-		</visual>
-		<collision>
-			<geometry>
-				<mesh filename="file:///home/marguedas/.ros/nao_meshes/meshes/V40/collision/LHip.ply" scale="0.001 0.001 0.001"/>
+				<mesh filename="package://nao_meshes/meshes/V40/visual/collada/LHip.dae" scale="0.1 0.1 0.1"/>
+			</geometry>
+		</visual>
+		<collision>
+			<geometry>
+				<mesh filename="package://nao_meshes/meshes/V40/visual/collada/LHip.dae" scale="0.1 0.1 0.1"/>
 			</geometry>
 		</collision>
@@ -59,10 +59,10 @@
 		<visual>
 			<geometry>
-				<mesh filename="file:///home/marguedas/.ros/nao_meshes/meshes/V40/visual/LThigh.obj" scale="0.001 0.001 0.001"/>
-			</geometry>
-		</visual>
-		<collision>
-			<geometry>
-				<mesh filename="file:///home/marguedas/.ros/nao_meshes/meshes/V40/collision/LThigh.ply" scale="0.001 0.001 0.001"/>
+				<mesh filename="package://nao_meshes/meshes/V40/visual/collada/LThigh.dae" scale="0.1 0.1 0.1"/>
+			</geometry>
+		</visual>
+		<collision>
+			<geometry>
+				<mesh filename="package://nao_meshes/meshes/V40/visual/collada/LThigh.dae" scale="0.1 0.1 0.1"/>
 			</geometry>
 		</collision>
@@ -83,10 +83,10 @@
 		<visual>
 			<geometry>
-				<mesh filename="file:///home/marguedas/.ros/nao_meshes/meshes/V40/visual/LTibia.obj" scale="0.001 0.001 0.001"/>
-			</geometry>
-		</visual>
-		<collision>
-			<geometry>
-				<mesh filename="file:///home/marguedas/.ros/nao_meshes/meshes/V40/collision/LTibia.ply" scale="0.001 0.001 0.001"/>
+				<mesh filename="package://nao_meshes/meshes/V40/visual/collada/LTibia.dae" scale="0.1 0.1 0.1"/>
+			</geometry>
+		</visual>
+		<collision>
+			<geometry>
+				<mesh filename="package://nao_meshes/meshes/V40/visual/collada/LTibia.dae" scale="0.1 0.1 0.1"/>
 			</geometry>
 		</collision>
@@ -107,10 +107,10 @@
 		<visual>
 			<geometry>
-				<mesh filename="file:///home/marguedas/.ros/nao_meshes/meshes/V40/visual/l_ankle.obj" scale="0.001 0.001 0.001"/>
-			</geometry>
-		</visual>
-		<collision>
-			<geometry>
-				<mesh filename="file:///home/marguedas/.ros/nao_meshes/meshes/V40/collision/l_ankle.ply" scale="0.001 0.001 0.001"/>
+				<mesh filename="package://nao_meshes/meshes/V40/visual/collada/l_ankle.dae" scale="0.1 0.1 0.1"/>
+			</geometry>
+		</visual>
+		<collision>
+			<geometry>
+				<mesh filename="package://nao_meshes/meshes/V40/visual/collada/l_ankle.dae" scale="0.1 0.1 0.1"/>
 			</geometry>
 		</collision>
@@ -129,4 +129,14 @@
 	</joint>
 	<link name="LFeet">
+		<visual>
+			<geometry>
+				<mesh filename="package://nao_meshes/meshes/V40/visual/collada/LFeet.dae" scale="0.1 0.1 0.1"/>
+			</geometry>
+		</visual>
+		<collision>
+			<geometry>
+				<mesh filename="package://nao_meshes/meshes/V40/visual/collada/LFeet.dae" scale="0.1 0.1 0.1"/>
+			</geometry>
+		</collision>
 		<inertial>
 			<mass value="0.16184"/>
@@ -145,10 +155,10 @@
 		<visual>
 			<geometry>
-				<mesh filename="file:///home/marguedas/.ros/nao_meshes/meshes/V40/visual/RPelvis.obj" scale="0.001 0.001 0.001"/>
-			</geometry>
-		</visual>
-		<collision>
-			<geometry>
-				<mesh filename="file:///home/marguedas/.ros/nao_meshes/meshes/V40/collision/RPelvis.ply" scale="0.001 0.001 0.001"/>
+				<mesh filename="package://nao_meshes/meshes/V40/visual/collada/RPelvis.dae" scale="0.1 0.1 0.1"/>
+			</geometry>
+		</visual>
+		<collision>
+			<geometry>
+				<mesh filename="package://nao_meshes/meshes/V40/visual/collada/RPelvis.dae" scale="0.1 0.1 0.1"/>
 			</geometry>
 		</collision>
@@ -169,10 +179,10 @@
 		<visual>
 			<geometry>
-				<mesh filename="file:///home/marguedas/.ros/nao_meshes/meshes/V40/visual/RHip.obj" scale="0.001 0.001 0.001"/>
-			</geometry>
-		</visual>
-		<collision>
-			<geometry>
-				<mesh filename="file:///home/marguedas/.ros/nao_meshes/meshes/V40/collision/RHip.ply" scale="0.001 0.001 0.001"/>
+				<mesh filename="package://nao_meshes/meshes/V40/visual/collada/RHip.dae" scale="0.1 0.1 0.1"/>
+			</geometry>
+		</visual>
+		<collision>
+			<geometry>
+				<mesh filename="package://nao_meshes/meshes/V40/visual/collada/RHip.dae" scale="0.1 0.1 0.1"/>
 			</geometry>
 		</collision>
@@ -193,10 +203,10 @@
 		<visual>
 			<geometry>
-				<mesh filename="file:///home/marguedas/.ros/nao_meshes/meshes/V40/visual/RThigh.obj" scale="0.001 0.001 0.001"/>
-			</geometry>
-		</visual>
-		<collision>
-			<geometry>
-				<mesh filename="file:///home/marguedas/.ros/nao_meshes/meshes/V40/collision/RThigh.ply" scale="0.001 0.001 0.001"/>
+				<mesh filename="package://nao_meshes/meshes/V40/visual/collada/RThigh.dae" scale="0.1 0.1 0.1"/>
+			</geometry>
+		</visual>
+		<collision>
+			<geometry>
+				<mesh filename="package://nao_meshes/meshes/V40/visual/collada/RThigh.dae" scale="0.1 0.1 0.1"/>
 			</geometry>
 		</collision>
@@ -217,10 +227,10 @@
 		<visual>
 			<geometry>
-				<mesh filename="file:///home/marguedas/.ros/nao_meshes/meshes/V40/visual/RTibia.obj" scale="0.001 0.001 0.001"/>
-			</geometry>
-		</visual>
-		<collision>
-			<geometry>
-				<mesh filename="file:///home/marguedas/.ros/nao_meshes/meshes/V40/collision/RTibia.ply" scale="0.001 0.001 0.001"/>
+				<mesh filename="package://nao_meshes/meshes/V40/visual/collada/RTibia.dae" scale="0.1 0.1 0.1"/>
+			</geometry>
+		</visual>
+		<collision>
+			<geometry>
+				<mesh filename="package://nao_meshes/meshes/V40/visual/collada/RTibia.dae" scale="0.1 0.1 0.1"/>
 			</geometry>
 		</collision>
@@ -241,10 +251,10 @@
 		<visual>
 			<geometry>
-				<mesh filename="file:///home/marguedas/.ros/nao_meshes/meshes/V40/visual/r_ankle.obj" scale="0.001 0.001 0.001"/>
-			</geometry>
-		</visual>
-		<collision>
-			<geometry>
-				<mesh filename="file:///home/marguedas/.ros/nao_meshes/meshes/V40/collision/r_ankle.ply" scale="0.001 0.001 0.001"/>
+				<mesh filename="package://nao_meshes/meshes/V40/visual/collada/r_ankle.dae" scale="0.1 0.1 0.1"/>
+			</geometry>
+		</visual>
+		<collision>
+			<geometry>
+				<mesh filename="package://nao_meshes/meshes/V40/visual/collada/r_ankle.dae" scale="0.1 0.1 0.1"/>
 			</geometry>
 		</collision>
@@ -263,4 +273,14 @@
 	</joint>
 	<link name="RFeet">
+		<visual>
+			<geometry>
+				<mesh filename="package://nao_meshes/meshes/V40/visual/collada/RFeet.dae" scale="0.1 0.1 0.1"/>
+			</geometry>
+		</visual>
+		<collision>
+			<geometry>
+				<mesh filename="package://nao_meshes/meshes/V40/visual/collada/RFeet.dae" scale="0.1 0.1 0.1"/>
+			</geometry>
+		</collision>
 		<inertial>
 			<mass value="0.16184"/>

File: outputs/naoOuttorso.xacro (robot description, xacro)
@@ -10,10 +10,10 @@
 		<visual>
 			<geometry>
-				<mesh filename="file:///home/marguedas/.ros/nao_meshes/meshes/V40/visual/collada/torso.dae" scale="0.1 0.1 0.1"/>
+				<mesh filename="package://nao_meshes/meshes/V40/visual/collada/torso.dae" scale="0.1 0.1 0.1"/>
 			</geometry>
 		</visual>
 		<collision>
 			<geometry>
-				<mesh filename="file:///home/marguedas/.ros/nao_meshes/meshes/V40/visual/collada/torso.dae" scale="0.1 0.1 0.1"/>
+				<mesh filename="package://nao_meshes/meshes/V40/visual/collada/torso.dae" scale="0.1 0.1 0.1"/>
 			</geometry>
 		</collision>
